Commit message: Aktualny stan

File: src/mechanical/rov_description/xacro/bluerov2.urdf.xacro (robot description, xacro)
@@ -25,5 +25,5 @@
   <xacro:property name="CoG_X" value="0"/>
   <xacro:property name="CoG_Y" value="0"/>
-  <xacro:property name="CoG_Z" value="0.08"/>
+  <xacro:property name="CoG_Z" value="0.072"/>
   <xacro:property name="CoG" value="${CoG_X} ${CoG_Y} ${CoG_Z}"/>
   <xacro:macro name='CoG_origin' params="X Y Z rpy" >

File: src/mechanical/rov_description/xacro/new_robot.urdf.xacro (robot description, xacro)
@@ -58,67 +58,67 @@
   </link>
   <!-- Thruster origins -->
-  <xacro:property name="front_right_origin">
-    <!-- <origin xyz="0.1355 0.1 0.0725" rpy="0 0 -0.7853981634"/> -->
-    <!-- <origin xyz="0.1355 0.1 -0.0725" rpy="${PI} 0 -0.7853981634"/> -->
-    <xacro:CoG_origin X="0.149471" Y="0.189471" Z="0.013" rpy="0 0 ${-PI/4}"/>
+    <xacro:property name="dive_rear_left_origin">
+    <!-- <origin xyz="-0.12 -0.218 0.0" rpy="0 -1.5707963268 0"/> -->
+    <!-- <origin xyz="-0.12 -0.218 0.0" rpy="${PI} -1.5707963268 0"/> -->
+    <xacro:CoG_origin X="-0.28325" Y="-0.20925" Z="0.00575" rpy="${PI} -1.5707963268 0"/>
+    </xacro:property>
+    <xacro:property name="rear_left_origin">
+    <!-- <origin xyz="-0.1475 -0.1 0.0725" rpy="0 0 2.3561944902"/> -->
+    <!-- <origin xyz="-0.1475 -0.1 -0.0725" rpy="${PI} 0 2.3561944902"/> -->
+    <xacro:CoG_origin X="-0.1568" Y="-0.18205" Z="0.008" rpy="0 0 2.3561944902"/>
   </xacro:property>
   <xacro:property name="front_left_origin">
     <!-- <origin xyz="0.1355 -0.1 0.0725" rpy="0 0 0.7853981634"/> -->
     <!-- <origin xyz="0.1355 -0.1 -0.0725" rpy="${PI} 0 0.7853981634"/> -->
-    <xacro:CoG_origin X="0.149471" Y="-0.189471" Z="0.013" rpy="0 0 ${PI/4}"/>
+    <xacro:CoG_origin X="0.1568" Y="-0.18205" Z="0.008" rpy="0 0 ${PI/4}"/>
+  </xacro:property>
+  <xacro:property name="dive_front_left_origin">
+    <!-- <origin xyz="0.12 -0.218 0.0" rpy="0 -1.5707963268 0"/> -->
+    <!-- <origin xyz="0.12 -0.218 0.0" rpy="${PI} -1.5707963268 0"/> -->
+    <xacro:CoG_origin X="0.28325" Y="-0.20925" Z="0.00575" rpy="${PI} 1.5707963268 0"/>
+  </xacro:property>
+  <xacro:property name="dive_rear_right_origin">
+    <!-- <origin xyz="-0.12 0.218 0.0" rpy="0 -1.5707963268 0"/> -->
+    <!-- <origin xyz="-0.12 0.218 0.0" rpy="${PI} -1.5707963268 0"/> -->
+    <xacro:CoG_origin X="-0.28325" Y="0.20925" Z="0.00575" rpy="${PI} 1.5707963268 0"/>
   </xacro:property>
   <xacro:property name="rear_right_origin">
     <!-- <origin xyz="-0.1475 0.1 0.0725" rpy="0 0 -2.3561944902"/> -->
     <!-- <origin xyz="-0.1475 0.1 -0.0725" rpy="${PI} 0 -2.3561944902"/> -->
-    <xacro:CoG_origin X="-0.149471" Y="0.189471" Z="0.013" rpy="0 0 -2.3561944902"/>
+    <xacro:CoG_origin X="-0.1568" Y="0.18205" Z="0.008" rpy="0 0 -2.3561944902"/>
   </xacro:property>
-  <xacro:property name="rear_left_origin">
-    <!-- <origin xyz="-0.1475 -0.1 0.0725" rpy="0 0 2.3561944902"/> -->
-    <!-- <origin xyz="-0.1475 -0.1 -0.0725" rpy="${PI} 0 2.3561944902"/> -->
-    <xacro:CoG_origin X="-0.149471" Y="-0.189471" Z="0.013" rpy="0 0 2.3561944902"/>
+  <xacro:property name="front_right_origin">
+    <!-- <origin xyz="0.1355 0.1 0.0725" rpy="0 0 -0.7853981634"/> -->
+    <!-- <origin xyz="0.1355 0.1 -0.0725" rpy="${PI} 0 -0.7853981634"/> -->
+    <xacro:CoG_origin X="0.1568" Y="0.18205" Z="0.008" rpy="0 0 ${-PI/4}"/>
   </xacro:property>
   <xacro:property name="dive_front_right_origin">
     <!-- <origin xyz="0.12 0.218 0.0" rpy="0 -1.5707963268 0"/> -->
     <!-- <origin xyz="0.12 0.218 0.0" rpy="${PI} -1.5707963268 0"/> -->
-    <xacro:CoG_origin X="0.26325" Y="0.20925" Z="0.0075" rpy="${PI} -1.5707963268 0"/>
-  </xacro:property>
-  <xacro:property name="dive_front_left_origin">
-    <!-- <origin xyz="0.12 -0.218 0.0" rpy="0 -1.5707963268 0"/> -->
-    <!-- <origin xyz="0.12 -0.218 0.0" rpy="${PI} -1.5707963268 0"/> -->
-    <xacro:CoG_origin X="0.26325" Y="-0.20925" Z="0.0075" rpy="${PI} -1.5707963268 0"/>
-  </xacro:property>
-  <xacro:property name="dive_rear_right_origin">
-    <!-- <origin xyz="-0.12 0.218 0.0" rpy="0 -1.5707963268 0"/> -->
-    <!-- <origin xyz="-0.12 0.218 0.0" rpy="${PI} -1.5707963268 0"/> -->
-    <xacro:CoG_origin X="-0.26325" Y="0.20925" Z="0.0075" rpy="${PI} -1.5707963268 0"/>
-  </xacro:property>
-  <xacro:property name="dive_rear_left_origin">
-    <!-- <origin xyz="-0.12 -0.218 0.0" rpy="0 -1.5707963268 0"/> -->
-    <!-- <origin xyz="-0.12 -0.218 0.0" rpy="${PI} -1.5707963268 0"/> -->
-    <xacro:CoG_origin X="-0.26325" Y="-0.20925" Z="0.0075" rpy="${PI} -1.5707963268 0"/>
+    <xacro:CoG_origin X="0.28325" Y="0.20925" Z="0.00575" rpy="${PI} -1.5707963268 0"/>
   </xacro:property>
   <!-- Attach thrusters to the base_link -->
-  <xacro:t200 name="t1" side="right">
+  <xacro:t200 name="t7" side="right">
     <xacro:insert_block name="front_right_origin"/>
   </xacro:t200>
-  <xacro:t200 name="t2" side="left">
+  <xacro:t200 name="t3" side="left">
     <xacro:insert_block name="front_left_origin"/>
   </xacro:t200>
-  <xacro:t200 name="t3" side="right">
+  <xacro:t200 name="t6" side="right">
     <xacro:insert_block name="rear_right_origin"/>
   </xacro:t200>
-  <xacro:t200 name="t4" side="left">
+  <xacro:t200 name="t2" side="left">
     <xacro:insert_block name="rear_left_origin"/>
   </xacro:t200>
-  <xacro:t200 name="t5" side="right">
+  <xacro:t200 name="t8" side="right">
     <xacro:insert_block name="dive_front_right_origin"/>
   </xacro:t200>
-  <xacro:t200 name="t6" side="left">
+  <xacro:t200 name="t4" side="left">
     <xacro:insert_block name="dive_front_left_origin"/>
   </xacro:t200>
-  <xacro:t200 name="t7" side="right">
+  <xacro:t200 name="t5" side="right">
     <xacro:insert_block name="dive_rear_right_origin"/>
   </xacro:t200>
-  <xacro:t200 name="t8" side="left">
+  <xacro:t200 name="t1" side="left">
     <xacro:insert_block name="dive_rear_left_origin"/>
   </xacro:t200>
